File: tank/turret_board/turret_board.kicad_pcb (KiCad board)
At the start: 2 copper layers, 38 x 38.7 mm, 47 parts, among them J1 Conn_01x02_Male, J2 Conn_01x04_Male, J3 Conn_01x03_Male, J4 Conn_01x02_Male, J5 Conn_01x02_Male, Q1 2N3904, Q2 2N3904, U1 KA378R33, U2 pixart_ir, Y1 Crystal_4pin

Commit message: revisions
Parts:
- removed Beacon1: CONN_01X02, Connector_JST:JST_EH_B2B-EH-A_1x02_P2.50mm_Vertical
- removed the C1 at (265.7, 120.4)
- removed C3: CP, Capacitors_THT:CP_Radial_D5.0mm_P2.00mm
- removed C3: C, custom:CP_Radial_D4.0mm_P2.00mm
- removed C5: C, Capacitors_THT:C_Disc_D3.0mm_W1.6mm_P2.50mm
- removed D1, D2, D3: D, Diodes_THT:D_T-1_P5.08mm_Horizontal
- removed D1, D2, D3: D-Device, custom:D_A-405_P7.62mm_Horizontal
- removed G***: LOGO, modules:Tank
- removed IRRx: CONN_01X03, Connector_JST:JST_EH_B3B-EH-A_1x03_P2.50mm_Vertical
- removed Power: Conn_01x02_Male, JST:JST_EH_B02B-EH-A_02x2.50mm_Straight
- removed the Q1 at (272.2, 109.9)
- removed Q2: 2N3904, TO_SOT_Packages_THT:TO-92_Inline_Narrow_Oval
- removed Q2: 2N3904, custom:TO-92
- removed the R2 at (241.6, 126.1)
- removed R5, R9: R, Resistors_THT:R_Axial_DIN0207_L6.3mm_D2.5mm_P7.62mm_Horizontal
- removed R5: R, custom:R_Axial_DIN0207_L6.3mm_D2.5mm_P7.62mm_Horizontal
- removed R8: R, Resistor_THT:R_Axial_DIN0207_L6.3mm_D2.5mm_P7.62mm_Horizontal
- removed REF** (x4): MountingHole_2.2mm_M2, Mounting_Holes:MountingHole_2.2mm_M2
- removed SigIn1: CONN_01X04, Connector_JST:JST_EH_B4B-EH-A_1x04_P2.50mm_Vertical
- removed Tx1: TX, Connector_JST:JST_EH_B2B-EH-A_1x02_P2.50mm_Vertical
- removed the U1 at (237.0, 114.8)
- removed the U2 at (230.1, 103.7)
- removed the Y1 at (239.7, 105.9)
- C1: value CP -> C_Small; footprint Capacitors_THT:CP_Radial_D5.0mm_P2.00mm -> custom:C_Disc_D4.7mm_W2.5mm_P5.00mm
- C1: footprint Capacitor_THT:C_Disc_D4.7mm_W2.5mm_P5.00mm -> custom:C_Disc_D4.7mm_W2.5mm_P5.00mm
- C2: value C_Small -> C; footprint custom:C_Disc_D4.7mm_W2.5mm_P5.00mm -> custom:CP_Radial_D4.0mm_P2.00mm
- Q1: footprint TO_SOT_Packages_THT:TO-92_Inline_Narrow_Oval -> custom:TO-92
- R2: footprint Resistors_THT:R_Axial_DIN0207_L6.3mm_D2.5mm_P7.62mm_Horizontal -> custom:R_Axial_DIN0207_L6.3mm_D2.5mm_P7.62mm_Horizontal
- U1: footprint TO_SOT_Packages_THT:TO-220-4_Vertical -> custom:LM317T
- U2: footprint modules:pixart_ir -> custom:pixart_ir
- Y1: footprint Tank:ECS-100AX -> custom:ECS-100AX
- moved R1 54.1 mm to (203.0, 125.6)
- moved J3 49.5 mm to (205.0, 120.3)
- moved R4 45.6 mm to (217.6, 113.9)
- moved J4 41.3 mm to (217.0, 124.4)
- moved J1 38.6 mm to (230.3, 114.5)
- moved J5 38.0 mm to (227.8, 120.3)
- moved R3 30.1 mm to (215.1, 119.8)
- moved J2 28.3 mm to (205.0, 114.5)
- moved C2 27.5 mm to (224.9, 126.3)
Connections:
- C1 pad 1: 5V -> Net-(C1-Pad1)
- C2 pad 1: Net-(C2-Pad1) -> 3.3V
- J5 pad 2: GND -> 5V
- Q1 pad 2: Net-(D3-Pad1) -> IRSig
- Q1 pad 3: Net-(D2-Pad1) -> Net-(Q1-Pad3)
- R1 pad 1: Net-(Q2-Pad2) -> IRTx
- R1 pad 2: Net-(C2-Pad1) -> Net-(Q1-Pad3)
- R2 pad 1: Net-(Q2-Pad2) -> IRTx
- R2 pad 2: Net-(C5-Pad1) -> Net-(Q1-Pad3)
- R3 pad 1: IRTx -> 5V
- R3 pad 2: Net-(D1-Pad2) -> Beacon
- R4 pad 1: 5V -> 3.3V
- R4 pad 2: Beacon -> RESET
- U2 pad 4: Net-(U2-Pad4) -> unconnected-(U2-Pad4)
- Y1 pad 1: Net-(Y1-Pad1) -> unconnected-(Y1-Pad1)
Routing:
- net Net-(C1-Pad1): track 31.4 -> 85.1 mm
- net 5V: track 53.7 -> 0.00 mm
- net IRSig: track 33.8 -> 0.00 mm
- net IRRx: track 45.4 -> 77.4 mm
- net Net-(Q1-Pad3): track 0.00 -> 24.3 mm
- net 3.3V: track 46.3 -> 26.6 mm
- net RESET: track 24.0 -> 4.31 mm
- net IRTx: track 12.0 -> 26.7 mm
- net Net-(Q2-Pad2): track 14.8 -> 0.00 mm
- net Net-(D2-Pad1): track 22.7 -> 10.1 mm
- net Net-(C5-Pad1): track 11.7 -> 0.00 mm
- net SDA: track 28.5 -> 17.3 mm
- net SLC: track 32.7 -> 21.5 mm
- net Net-(D3-Pad1): track 25.9 -> 15.1 mm
Other:
- board size 38 x 38.7 mm -> 36 x 39 mm
- net class Default removed

Commit message: turret board v0.8
Parts:
- removed the C1 at (192.5, 102.2)
- removed the C1 at (197.2, 100.5)
- removed J1, J4, J5: Conn_01x02_Male, custom:JST_EH_B2B-EH-A_1x02_P2.50mm_Vertical
- removed J2: Conn_01x04_Male, custom:JST_EH_B4B-EH-A_1x04_P2.50mm_Vertical
- removed J3: Conn_01x03_Male, custom:JST_EH_B3B-EH-A_1x03_P2.50mm_Vertical
- removed R4: R, custom:R_Axial_DIN0207_L6.3mm_D2.5mm_P7.62mm_Horizontal
- added Beacon1: Conn_01x02_Male, custom:JST_EH_B2B-EH-A_1x02_P2.50mm_Vertical, F.Cu at (218.0, 97.0)
- added C1: C_Small, Capacitor_THT:CP_Radial_D4.0mm_P2.00mm, F.Cu at (211.0, 115.0)
- added IRRx1: Conn_01x03_Male, custom:JST_EH_B3B-EH-A_1x03_P2.50mm_Vertical, F.Cu at (184.4, 100.8)
- added IRTx1: Conn_01x02_Male, custom:JST_EH_B2B-EH-A_1x02_P2.50mm_Vertical, F.Cu at (194.8, 121.3)
- added Power1: Conn_01x02_Male, custom:JST_EH_B2B-EH-A_1x02_P2.50mm_Vertical, F.Cu at (184.2, 114.2)
- added REF**: MountingHole_2.2mm_M2, MountingHole:MountingHole_2.2mm_M2, F.Cu at (219.0, 89.5)
- added REF**: MountingHole_2.2mm_M2, MountingHole:MountingHole_2.2mm_M2, F.Cu at (219.0, 120.5)
- added REF**: MountingHole_2.2mm_M2, MountingHole:MountingHole_2.2mm_M2, F.Cu at (183.5, 89.5)
- added REF**: MountingHole_2.2mm_M2, MountingHole:MountingHole_2.2mm_M2, F.Cu at (183.5, 120.5)
- added SigIn1: Conn_01x04_Male, custom:JST_EH_B4B-EH-A_1x04_P2.50mm_Vertical, F.Cu at (218.0, 107.5)
- C2: value C -> C_Polarized_Small; footprint custom:CP_Radial_D4.0mm_P2.00mm -> Capacitor_THT:C_Disc_D4.7mm_W2.5mm_P5.00mm
- U1: value KA378R33 -> LD1117; footprint custom:LM317T -> custom:LD1117
- moved R1 26.3 mm to (189.5, 103.0), turned to -90 degrees
- moved R2 20.6 mm to (205.2, 122.5), turned to 0 degrees
- moved C2 20.2 mm to (206.5, 118.0), turned to 90 degrees
- moved U1 16.7 mm to (202.0, 113.5), turned to -90 degrees
- moved R3 15.5 mm to (212.5, 104.5), turned to 90 degrees
- moved Y1 14.8 mm to (193.9, 98.7), turned to 0 degrees
- moved Q1 3.98 mm to (194.2, 111.9), turned to -90 degrees
Connections:
- R2 pad 1: IRTx -> 5V
- R2 pad 2: Net-(Q1-Pad3) -> Beacon
- R3 pad 1: 5V -> 3.3V
- R3 pad 2: Beacon -> RESET
- U1 pad 1: Net-(C1-Pad1) -> GND
- U1 pad 3: GND -> Net-(C1-Pad1)
Routing:
- net 5V: track 0.00 -> 81.5 mm
- net Net-(C1-Pad1): track 85.1 -> 31.6 mm
- net IRRx: track 77.4 -> 36.3 mm
- net 3.3V: track 26.6 -> 53.2 mm
- net IRSig: track 0.00 -> 23.8 mm
- net Net-(Q1-Pad3): track 24.3 -> 6.28 mm
- net GND: track 99.8 -> 83.6 mm
- net Net-(D3-Pad1): track 15.1 -> 0.00 mm
- net SLC: track 21.5 -> 35.9 mm
- net SDA: track 17.3 -> 28.6 mm
- net Net-(D2-Pad1): track 10.1 -> 0.00 mm
- net IRTx: track 26.7 -> 20.4 mm
- net RESET: track 4.31 -> 9.55 mm
- net Net-(U2-Pad7): track 6.70 -> 10.5 mm
- net Beacon: track 31.6 -> 33.2 mm
Other:
- board size 36 x 39 mm -> 40.5 x 37.5 mm
- board text added: "Turret Board v0.8 Laser Tag Robot Tank M.I.A.R. Labs nick.groesz@gmail.com"
- board text removed: "Turret Board v0.7 Laser Tag Robot Tank M.I.A.R. Labs nick.groesz@gmail.com"

Commit message: turret board v0.9
Parts:
- removed Q1: 2N3904, custom:TO-92
- removed the REF** at (219.0, 89.5)
- removed the REF** at (219.0, 120.5)
- removed the REF** at (183.5, 89.5)
- removed the REF** at (183.5, 120.5)
- added REF**: MountingHole_2.2mm_M2, MountingHole:MountingHole_2.2mm_M2, F.Cu at (183.5, 120.6)
- added REF**: MountingHole_2.2mm_M2, MountingHole:MountingHole_2.2mm_M2, F.Cu at (219.0, 89.5)
- added REF**: MountingHole_2.2mm_M2, MountingHole:MountingHole_2.2mm_M2, F.Cu at (219.0, 120.6)
- added REF**: MountingHole_2.2mm_M2, MountingHole:MountingHole_2.2mm_M2, F.Cu at (183.5, 89.6)
- moved R1 12.9 mm to (197.0, 113.5), turned to 180 degrees
- moved SigIn1 6.52 mm to (218.5, 114.0), turned to 90 degrees
- moved IRTx1 3.52 mm to (191.2, 121.7), turned to 0 degrees
- moved Beacon1 2.55 mm to (218.5, 99.5), turned to 90 degrees
- moved Y1 2.55 mm to (191.4, 98.2)
- moved IRRx1 2.29 mm to (184.0, 98.5), turned to -90 degrees
- moved Power1 1.76 mm to (184.0, 112.5), turned to -90 degrees
Connections:
- net IRRx renamed /IRRx
- net RESET renamed Net-(R3-Pad2)
- Beacon1 pad 1: Beacon -> GND
- Beacon1 pad 2: 5V -> Net-(Beacon1-Pad2)
- C1 pad 1: Net-(C1-Pad1) -> 5V
- IRTx1 pad 1: 5V -> GND
- IRTx1 pad 2: IRTx -> /IRTx
- Power1 pad 1: Net-(C1-Pad1) -> 5V
- R1 pad 1: IRTx -> Net-(R1-Pad1)
- R1 pad 2: Net-(Q1-Pad3) -> /IRTx
- R2 pad 2: Beacon -> Net-(Beacon1-Pad2)
- SigIn1 pad 2: IRSig -> Net-(R1-Pad1)
- U1 pad 3: Net-(C1-Pad1) -> 5V
Routing:
- net 5V: track 81.5 -> 44.4 mm
- net Beacon: track 33.2 -> 0.00 mm
- net Net-(C1-Pad1): track 31.6 -> 0.00 mm
- net Net-(Beacon1-Pad2): track 0.00 -> 29.5 mm
- net IRSig: track 23.8 -> 0.00 mm
- net Net-(R1-Pad1): track 0.00 -> 22.3 mm
- net IRTx: track 20.4 -> 0.00 mm
- net /IRTx: track 0.00 -> 10.0 mm
- net SLC: track 35.9 -> 26.7 mm
- net /IRRx: track 36.3 -> 45.4 mm
- net GND: track 83.6 -> 91.8 mm
- net Net-(Q1-Pad3): track 6.28 -> 0.00 mm
- net SDA: track 28.6 -> 25.3 mm
- net Net-(U2-Pad7): track 10.5 -> 8.99 mm
- net 3.3V: track 53.2 -> 53.6 mm, vias 0 -> 1
Other:
- board text added: "Turret Board v0.9 Laser Tag Robot Tank M.I.A.R. Labs nick.groesz@gmail.com"
- board text removed: "Turret Board v0.8 Laser Tag Robot Tank M.I.A.R. Labs nick.groesz@gmail.com"
