File: tank/turret_board/turret_board.kicad_pcb (KiCad board)
At the start: 2 copper layers, 40.5 x 37.5 mm, 17 parts, among them U1 LD1117, U2 pixart_ir, Y1 Crystal_4pin

Commit message: Turret Board v0.10: add connector for second I²C device
Parts:
- added SigIn2: Conn_01x04_Male, custom:JST_EH_B4B-EH-A_1x04_P2.50mm_Vertical, F.Cu at (205.6, 121.7)
- moved R2 18.0 mm to (188.4, 116.1)
- moved C1 2.80 mm to (210.9, 112.2)
- moved R1 1.97 mm to (196.0, 111.8)
- moved C2 1.92 mm to (206.2, 116.1)
- moved U1 1.58 mm to (201.1, 112.2)
Routing:
- net SLC: track 26.7 -> 49.9 mm
- net SDA: track 25.3 -> 43.8 mm
- net Net-(Beacon1-Pin_2): track 29.5 -> 47.8 mm
- net GND: track 91.8 -> 108.7 mm
- net Net-(SigIn1-Pin_2): track 22.3 -> 34.0 mm, vias 0 -> 1
- net 3.3V: track 53.6 -> 60.8 mm, vias 1 -> 0
- net /IRRx: track 45.4 -> 41.8 mm
- net 5V: track 44.4 -> 42.1 mm
- net /IRTx: track 10.0 -> 12.1 mm
Other:
- board text added: "R1"
- board text added: "R2"
- board text added: "Turret Board v0.10 Laser Tag Robot Tank M.I.A.R. Labs nick.groesz@gmail.com"
- board text removed: "Turret Board v0.9 Laser Tag Robot Tank M.I.A.R. Labs nick.groesz@gmail.com"

Commit message: minor changes for turret board v0.11
Parts:
- removed REF** (x4): MountingHole_2.2mm_M2, MountingHole:MountingHole_2.2mm_M2
- removed SigIn2: Conn_01x04_Male, custom:JST_EH_B4B-EH-A_1x04_P2.50mm_Vertical
- added Distance1: Conn_01x04_Male, custom:JST_EH_B4B-EH-A_1x04_P2.50mm_Vertical, F.Cu at (205.7, 121.7)
- added H1: MountingHole, MountingHole:MountingHole_2.2mm_M2, F.Cu at (183.6, 120.6)
- added H2: MountingHole, MountingHole:MountingHole_2.2mm_M2, F.Cu at (218.9, 120.6)
- added H3: MountingHole, MountingHole:MountingHole_2.2mm_M2, F.Cu at (183.6, 89.6)
- added H4: MountingHole, MountingHole:MountingHole_2.2mm_M2, F.Cu at (219.0, 89.5)
