File: tank/turret_board/turret_board.kicad_sch (KiCad schematic)
At the start: 15 parts, among them J1 Conn_01x02_Male, J2 Conn_01x04_Male, J3 Conn_01x03_Male, J4 Conn_01x02_Male, J5 Conn_01x02_Male, Q1 2N3904, U1 KA378R33, U2 pixart_ir, Y1 Crystal_4pin

Commit message: turret board v0.8
Parts:
- removed C1: C_Small, custom:C_Disc_D4.7mm_W2.5mm_P5.00mm, symbol custom:C_Small
- removed C2: C, custom:CP_Radial_D4.0mm_P2.00mm, symbol custom:C
- removed R1: R, custom:R_Axial_DIN0207_L6.3mm_D2.5mm_P7.62mm_Horizontal, symbol custom:R
- removed U1: KA378R33, custom:LM317T, symbol custom:KA378R33
- added C1: C_Small, Capacitor_THT:CP_Radial_D4.0mm_P2.00mm, symbol Device:C_Small
- added C2: C_Polarized_Small, Capacitor_THT:C_Disc_D4.7mm_W2.5mm_P5.00mm, symbol Device:C_Polarized_Small
- added U1: LD1117, custom:LD1117, symbol custom:LD1117
- renumbered J5 to Beacon1, J3 to IRRx1, J4 to IRTx1, J1 to Power1, R2 to R1, R3 to R2, R4 to R3, J2 to SigIn1
Connections:
- net 3.3V: now also C2.1, U1.2 (VO)
- net GND: now also C1.2, C2.2, U1.1 (ADJ/GND)
- net at Power1.1 (Pin_1): now also C1.1, U1.3 (VI)
- no-connect marks 3 -> 2
Other:
- moved on the sheet: IRRx1, R3, SigIn1

Commit message: turret board v0.9
Parts:
- removed Q1: 2N3904, custom:TO-92, symbol custom:2N3904
Connections:
- net 5V: now also C1.1, Power1.1 (Pin_1), U1.3 (VI); no longer Beacon1.2 (Pin_2), IRTx1.1 (Pin_1)
- net GND: now also Beacon1.1 (Pin_1), IRTx1.1 (Pin_1)
- net IRTx: now also R1.2; no longer R1.1
- net Beacon: no longer names the net of R2.2
- net Beacon: now also Beacon1.2 (Pin_2); no longer Beacon1.1 (Pin_1)
- net IRSig: no longer names the net of SigIn1.2 (Pin_2)
- net IRSig: now also R1.1
- net RESET: no longer names the net of R3.2, U2.8 (RESET)
