File: tank/main_board/main_board.sch (KiCad schematic (older format))
At the start: 35 parts, among them J1 PowerIn, J10 Sonar2, J11 Programming Header, J12 SigOut, J16 PowerOut, J2 M2, J3 M1, J4 LEDs, J5 M3, J6 Spk, J7 Hall2, J8 Hall1, J9 Sonar1, Q1 2N3904, U1 L7805, U2 ATMEGA328P-PU, U3 SN74HC595, U4 TB6612FNG, U5 TB6612FNG, Y1 Crystal

Commit message: tank main board version 0.5: - separate power supplies - sonar connectors are now bump encoders - removed PWN line for turret motor
Parts:
- removed J2: M2, Custom:TerminalBlock_4UCON_19963_02x4.5mm_Straight, symbol main_board-rescue:Conn_01x02
- removed J3: M1, Custom:TerminalBlock_4UCON_19963_02x4.5mm_Straight, symbol main_board-rescue:Conn_01x02
- removed J4: LEDs, Connectors_JST:JST_EH_B05B-EH-A_05x2.50mm_Straight, symbol main_board-rescue:Conn_01x05
- removed J5: M3, Custom:TerminalBlock_4UCON_19963_02x4.5mm_Straight, symbol main_board-rescue:Conn_01x02
- added J13: Encoder0, JST:JST_EH_B03B-EH-A_03x2.50mm_Straight, symbol main_board-rescue:Conn_01x03_Male
- added J14: Encoder1, JST:JST_EH_B03B-EH-A_03x2.50mm_Straight, symbol main_board-rescue:Conn_01x03_Male
- added J2: M1, JST:JST_EH_B02B-EH-A_02x2.50mm_Straight, symbol main_board-rescue:Conn_01x02_Male
- added J20: PowerMotor, JST:JST_EH_B02B-EH-A_02x2.50mm_Straight, symbol main_board-rescue:Conn_01x02_Male
- added J3: M2, JST:JST_EH_B02B-EH-A_02x2.50mm_Straight, symbol main_board-rescue:Conn_01x02_Male
- added J4: LEDs, JST:JST_EH_B04B-EH-A_04x2.50mm_Straight, symbol main_board-rescue:Conn_01x04_Male
- added J5: M0, JST:JST_EH_B02B-EH-A_02x2.50mm_Straight, symbol main_board-rescue:Conn_01x02_Male
- J10: value Sonar2 -> Bump1
- J9: value Sonar1 -> Bump0
Connections:
- net labels added: Bump0, Bump1, Encoder0, Encoder1, Gm, Vm
- net labels removed: 5V, LED3, M2PWM, Sonar0, Sonar1
- wire segments 122 -> 133
Changed lines of the file:
@@
 P 1850 3000
 F 0 "J9" H 1850 3200 50  0000 C CNN
-F 1 "Sonar1" H 1850 2800 50  0000 C CNN
+F 1 "Bump0" H 1850 2800 50  0000 C CNN
 F 2 "JST:JST_EH_B03B-EH-A_03x2.50mm_Straight" H 1850 3000 50  0001 C CNN
 F 3 "" H 1850 3000 50  0001 C CNN
@@
 P 1850 3500
 F 0 "J10" H 1850 3700 50  0000 C CNN
-F 1 "Sonar2" H 1850 3300 50  0000 C CNN
+F 1 "Bump1" H 1850 3300 50  0000 C CNN
 F 2 "JST:JST_EH_B03B-EH-A_03x2.50mm_Straight" H 1850 3500 50  0001 C CNN
 F 3 "" H 1850 3500 50  0001 C CNN
@@
 	-1   0    0    1
 $EndComp
-$Comp
-L main_board-rescue:Conn_01x02 J2
-U 1 1 59FE54C8
-P 10650 2500
-F 0 "J2" H 10650 2600 50  0000 C CNN
-F 1 "M2" H 10650 2300 50  0000 C CNN
-F 2 "Custom:TerminalBlock_4UCON_19963_02x4.5mm_Straight" H 10650 2500 50  0001 C CNN
-F 3 "" H 10650 2500 50  0001 C CNN
-	1    10650 2500
-	1    0    0    -1
-$EndComp
-$Comp
-L main_board-rescue:Conn_01x02 J3
-U 1 1 59FE55BC
-P 10600 1900
-F 0 "J3" H 10600 2000 50  0000 C CNN
-F 1 "M1" H 10600 1700 50  0000 C CNN
-F 2 "Custom:TerminalBlock_4UCON_19963_02x4.5mm_Straight" H 10600 1900 50  0001 C CNN
-F 3 "" H 10600 1900 50  0001 C CNN
-	1    10600 1900
-	1    0    0    -1
-$EndComp
 NoConn ~ 2400 4350
 $Comp
@@
 IRRx
 Text GLabel 5100 750  0    60   Input ~ 0
-5V
+9V
 $Comp
 L main_board-rescue:L7805 U1
@@
 SER
 Text GLabel 7650 1900 0    60   Input ~ 0
-5V
+Vm
 Wire Wire Line
 	8650 1900 8650 2000
@@
 Text GLabel 8650 2600 0    60   Input ~ 0
 4.5V
-Text GLabel 8650 2400 0    60   Input ~ 0
-GND
 Text GLabel 8650 2700 0    60   Input ~ 0
 M0+
@@
 Connection ~ 7750 2200
 Text GLabel 7600 2200 0    60   Input ~ 0
-GND
+Gm
 Text GLabel 5850 4250 2    60   Input ~ 0
 Hall0
@@
 	5750 4400 5850 4400
 Text GLabel 5250 3450 2    60   Input ~ 0
-Sonar1
+Bump1
 Text GLabel 2050 3600 2    60   Input ~ 0
-Sonar1
+Bump1
 Text GLabel 5250 3350 2    60   Input ~ 0
-Sonar0
+Bump0
 Text GLabel 2050 3100 2    60   Input ~ 0
-Sonar0
+Bump0
 Text GLabel 2100 2350 2    60   Input ~ 0
 Hall0
 Text GLabel 2050 2700 2    60   Input ~ 0
 Hall1
-$Comp
-L main_board-rescue:Conn_01x05 J4
-U 1 1 5A48A51B
-P 6900 1550
-F 0 "J4" H 6900 1850 50  0000 C CNN
-F 1 "LEDs" H 6900 1250 50  0000 C CNN
-F 2 "Connectors_JST:JST_EH_B05B-EH-A_05x2.50mm_Straight" H 6900 1550 50  0001 C CNN
-F 3 "" H 6900 1550 50  0001 C CNN
-	1    6900 1550
-	1    0    0    -1
-$EndComp
-Text GLabel 6700 1350 0    60   Input ~ 0
-5V
-Text GLabel 6700 1450 0    60   Input ~ 0
+Text GLabel 5500 1500 0    60   Input ~ 0
+4.5V
+Text GLabel 5500 1600 0    60   Input ~ 0
 LED0
-Text GLabel 6700 1550 0    60   Input ~ 0
+Text GLabel 5500 1700 0    60   Input ~ 0
 LED1
-Text GLabel 6700 1650 0    60   Input ~ 0
+Text GLabel 5500 1800 0    60   Input ~ 0
 LED2
-Text GLabel 6700 1750 0    60   Input ~ 0
-LED3
 Text GLabel 5250 2500 2    60   Input ~ 0
 M0PWM
@@
 M1PWM
 Text GLabel 5250 2700 2    60   Input ~ 0
-M2PWM
+Encoder0
 Text GLabel 5250 2400 2    60   Input ~ 0
 SER
@@
 LED2
 Text GLabel 5250 4600 2    60   Input ~ 0
-LED3
+Encoder1
 Text GLabel 8450 5450 2    60   Input ~ 0
 M2+
 Text GLabel 8450 5550 2    60   Input ~ 0
 M2-
-$Comp
-L main_board-rescue:Conn_01x02 J5
-U 1 1 5A48BFCF
-P 10600 3300
-F 0 "J5" H 10600 3400 50  0000 C CNN
-F 1 "M3" H 10600 3100 50  0000 C CNN
-F 2 "Custom:TerminalBlock_4UCON_19963_02x4.5mm_Straight" H 10600 3300 50  0001 C CNN
-F 3 "" H 10600 3300 50  0001 C CNN
-	1    10600 3300
-	1    0    0    -1
-$EndComp
 Wire Wire Line
 	10000 3300 10400 3300
@@
 	10100 3400 10400 3400
 Text GLabel 7650 3300 0    60   Input ~ 0
-5V
+Vm
 Wire Wire Line
 	7650 3300 7750 3300
@@
 Text GLabel 8650 4000 0    60   Input ~ 0
 4.5V
-Text GLabel 8650 3800 0    60   Input ~ 0
-GND
 Text GLabel 8650 4100 0    60   Input ~ 0
 M2+
@@
 Connection ~ 7750 3600
 Text GLabel 7600 3600 0    60   Input ~ 0
-GND
-Text GLabel 8650 4300 0    60   Input ~ 0
-M2PWM
+Gm
 NoConn ~ 8650 3500
 NoConn ~ 8650 3600
@@
 	1500 5850 1800 5850
 Wire Wire Line
-	2200 6150 2850 6150
+	2200 6150 2450 6150
 Wire Wire Line
 	2850 6150 3200 6150
@@
 Text GLabel 5850 4100 2    60   Input ~ 0
 Rx
+Wire Wire Line
+	3150 6850 3450 6850
+Wire Wire Line
+	3150 6950 3250 6950
+Text GLabel 3450 6850 2    50   Input ~ 0
+Vm
+Text GLabel 2950 6850 0    50   Input ~ 0
+Vm
+Text GLabel 2950 6950 0    50   Input ~ 0
+Gm
+$Comp
+L main_board-rescue:Conn_01x02_Male J20
+U 1 1 5E9AA91A
+P 2950 6850
+F 0 "J20" H 2950 6950 50  0000 C CNN
+F 1 "PowerMotor" H 2950 6650 50  0000 C CNN
+F 2 "JST:JST_EH_B02B-EH-A_02x2.50mm_Straight" H 2950 6850 50  0001 C CNN
+F 3 "" H 2950 6850 50  0001 C CNN
+	1    2950 6850
+	1    0    0    -1
+$EndComp
+Text GLabel 3450 6950 2    50   Input ~ 0
+Gm
+Wire Wire Line
+	2450 6150 2450 7200
+Wire Wire Line
+	2450 7200 3250 7200
+Wire Wire Line
+	3250 7200 3250 6950
+Connection ~ 2450 6150
+Wire Wire Line
+	2450 6150 2850 6150
+Connection ~ 3250 6950
+Wire Wire Line
+	3250 6950 3450 6950
+Wire Wire Line
+	8650 2400 7750 2400
+Wire Wire Line
+	7750 2400 7750 2200
+Wire Wire Line
+	8650 3800 7750 3800
+Wire Wire Line
+	7750 3800 7750 3600
+Text GLabel 8650 4300 0    60   Input ~ 0
+4.5V
+$Comp
+L main_board-rescue:Conn_01x03_Male J13
+U 1 1 5E9F4FF5
+P 1850 1100
+F 0 "J13" H 1958 1381 50  0000 C CNN
+F 1 "Encoder0" H 1958 1290 50  0000 C CNN
+F 2 "JST:JST_EH_B03B-EH-A_03x2.50mm_Straight" H 1850 1100 50  0001 C CNN
+F 3 "" H 1850 1100 50  0001 C CNN
+	1    1850 1100
+	1    0    0    -1
+$EndComp
+$Comp
+L main_board-rescue:Conn_01x03_Male J14
+U 1 1 5EA0741C
+P 1850 1550
+F 0 "J14" H 1958 1831 50  0000 C CNN
+F 1 "Encoder1" H 1958 1740 50  0000 C CNN
+F 2 "JST:JST_EH_B03B-EH-A_03x2.50mm_Straight" H 1850 1550 50  0001 C CNN
+F 3 "" H 1850 1550 50  0001 C CNN
+	1    1850 1550
+	1    0    0    -1
+$EndComp
+Text GLabel 2050 1000 2    60   Input ~ 0
+4.5V
+Text GLabel 2050 1450 2    60   Input ~ 0
+4.5V
+Text GLabel 2050 1100 2    60   Input ~ 0
+GND
+Text GLabel 2050 1550 2    60   Input ~ 0
+GND
+Text GLabel 2050 1200 2    60   Input ~ 0
+Encoder0
+Text GLabel 2050 1650 2    60   Input ~ 0
+Encoder1
+$Comp
+L main_board-rescue:Conn_01x04_Male J4
+U 1 1 5EA682FF
+P 5700 1700
+F 0 "J4" H 5700 1900 50  0000 C CNN
+F 1 "LEDs" H 5700 1400 50  0000 C CNN
+F 2 "JST:JST_EH_B04B-EH-A_04x2.50mm_Straight" H 5700 1700 50  0001 C CNN
+F 3 "" H 5700 1700 50  0001 C CNN
+	1    5700 1700
+	-1   0    0    1
+$EndComp
+$Comp
+L main_board-rescue:Conn_01x02_Male J2
+U 1 1 5E9835C0
+P 10600 2000
+F 0 "J2" H 10600 2100 50  0000 C CNN
+F 1 "M1" H 10600 1800 50  0000 C CNN
+F 2 "JST:JST_EH_B02B-EH-A_02x2.50mm_Straight" H 10600 2000 50  0001 C CNN
+F 3 "" H 10600 2000 50  0001 C CNN
+	1    10600 2000
+	-1   0    0    1
+$EndComp
+$Comp
+L main_board-rescue:Conn_01x02_Male J5
+U 1 1 5E98A5F8
+P 10650 2600
+F 0 "J5" H 10650 2700 50  0000 C CNN
+F 1 "M0" H 10650 2400 50  0000 C CNN
+F 2 "JST:JST_EH_B02B-EH-A_02x2.50mm_Straight" H 10650 2600 50  0001 C CNN
+F 3 "" H 10650 2600 50  0001 C CNN
+	1    10650 2600
+	-1   0    0    1
+$EndComp
+$Comp
+L main_board-rescue:Conn_01x02_Male J3
+U 1 1 5E98F9A1
+P 10600 3400
+F 0 "J3" H 10600 3500 50  0000 C CNN
+F 1 "M2" H 10600 3200 50  0000 C CNN
+F 2 "JST:JST_EH_B02B-EH-A_02x2.50mm_Straight" H 10600 3400 50  0001 C CNN
+F 3 "" H 10600 3400 50  0001 C CNN
+	1    10600 3400
+	-1   0    0    1
+$EndComp
 $EndSCHEMATC
