File: tank/main_board/main_board.sch (KiCad schematic (older format))
At the start: 38 parts, among them J1 PowerIn, J10 Bump1, J11 Programming Header, J12 SigOut, J13 Encoder0, J14 Encoder1, J16 PowerOut, J2 M1, J20 PowerMotor, J3 M2, J4 LEDs, J5 M0, J6 Spk, J7 Encoder3, J8 Encoder2, J9 Bump0, Q1 2N3904, U1 L7805, U2 ATMEGA328P-PU, U3 SN74HC595, U4 TB6612FNG, U5 TB6612FNG, Y1 Crystal

Commit message: main board 0.8 WIP
Parts:
- removed C6: C6, Capacitors_THT:C_Disc_D4.7mm_W2.5mm_P5.00mm, symbol main_board-rescue:C_Small
- added C7: C7, Capacitor_THT:C_Disc_D4.7mm_W2.5mm_P5.00mm, symbol main_board-rescue:C_Small
- C2, C8, C9: footprint Capacitors_THT:C_Disc_D4.7mm_W2.5mm_P5.00mm -> Capacitor_THT:C_Disc_D4.7mm_W2.5mm_P5.00mm
- C5: renamed from C7; footprint (none) -> Capacitor_THT:C_Disc_D4.7mm_W2.5mm_P5.00mm
- C6: renamed from C5; value C5 -> C6; footprint Capacitors_THT:C_Disc_D4.7mm_W2.5mm_P5.00mm -> Capacitor_THT:C_Disc_D4.7mm_W2.5mm_P5.00mm
- J8: renamed from J10; footprint JST:JST_EH_B03B-EH-A_03x2.50mm_Straight -> Connector_JST:JST_EH_B2B-EH-A_1x02_P2.50mm_Vertical
- renumbered J16 to J1, J20 to J10, J12 to J11, J6 to J12, J4 to J13, J2 to J14, J3 to J15, J5 to J16, J1 to J2, J13 to J3, J14 to J4, J8 to J5, J7 to J6, J9 to J7, J11 to J9, R11 to R1, R7 to R2, R6 to R3, R10 to R4
Connections:
- net 4.5V: now also J12.1 (Pin_1), J3.2 (Pin_2), J4.2 (Pin_2), J5.2 (Pin_2), J6.2 (Pin_2); no longer J3.1 (Pin_1), J4.1 (Pin_1), J5.1 (Pin_1), J6.1 (Pin_1)
- net 9V: no longer J12.1 (Pin_1)
- net Encoder0: now also J3.1 (Pin_1); no longer J3.3 (Pin_3)
- net Encoder1: now also J4.1 (Pin_1); no longer J4.3 (Pin_3)
- net Encoder2: now also J5.1 (Pin_1); no longer J5.3 (Pin_3)
- net Encoder3: now also J6.1 (Pin_1); no longer J6.3 (Pin_3)
- net GND: now also J3.3 (Pin_3), J4.3 (Pin_3), J5.3 (Pin_3), J6.3 (Pin_3), C7.2; no longer J3.2 (Pin_2), J4.2 (Pin_2), J5.2 (Pin_2), J6.2 (Pin_2)
- net at U2.10 ((PCINT7/XTAL2/TOSC2)PB7), Y1.1: now also C7.1
- no-connect marks 12 -> 8

Commit message: l293d version
Parts:
- removed C10, C11: CP, Capacitors_THT:CP_Radial_D4.0mm_P2.00mm, symbol main_board-rescue:CP
- removed C8, C9: C, Capacitor_THT:C_Disc_D4.7mm_W2.5mm_P5.00mm, symbol main_board-rescue:C
- removed Q1: 2N3904, TO_SOT_Packages_THT:TO-92_Molded_Narrow, symbol main_board-rescue:2N3904
- removed R1: R11, Resistors_THT:R_Axial_DIN0207_L6.3mm_D2.5mm_P7.62mm_Horizontal, symbol main_board-rescue:R
- removed U4, U5: TB6612FNG, Custom:TB6612FNG, symbol custom:TB6612FNG
- added C8: C_Small, Capacitor_THT:C_Disc_D4.7mm_W2.5mm_P5.00mm, symbol Device:C_Small
- added D1: D, Diode_THT:D_DO-35_SOD27_P2.54mm_Vertical_AnodeUp, symbol Device:D
- added R1: R, Resistor_THT:R_Axial_DIN0207_L6.3mm_D2.5mm_P7.62mm_Horizontal, symbol Device:R
- added U4, U5: L293D, Package_DIP:DIP-16_W7.62mm, symbol Driver_Motor:L293D
- J14: value M1 -> M0; footprint JST:JST_EH_B02B-EH-A_02x2.50mm_Straight -> Connector_JST:JST_EH_B2B-EH-A_1x02_P2.50mm_Vertical
- J15: value M2 -> M1; footprint JST:JST_EH_B02B-EH-A_02x2.50mm_Straight -> Connector_JST:JST_EH_B2B-EH-A_1x02_P2.50mm_Vertical
- J16: value M0 -> M2; footprint JST:JST_EH_B02B-EH-A_02x2.50mm_Straight -> Connector_JST:JST_EH_B2B-EH-A_1x02_P2.50mm_Vertical
- U1: symbol main_board-rescue:L7805 -> Regulator_Linear:L7805
Connections:
- net 4.5V: now also D1.1 (K), R1.1, U4.16 (VCC1), U5.16 (VCC1); no longer J12.1 (Pin_1)
- net GND: now also J12.1 (Pin_1), C8.2, U4.12 (GND), U4.13 (GND), U4.4 (GND), U4.5 (GND), U5.12 (GND), U5.13 (GND), U5.4 (GND), U5.5 (GND)
- net M0+: now also U4.2 (1A)
- net M0-: now also U4.7 (2A)
- net M0PWM: now also U4.1 (EN1,2)
- net M1+: now also U4.10 (3A)
- net M1-: now also U4.15 (4A)
- net M1PWM: now also U4.9 (EN3,4)
- net M2+: now also U5.2 (1A)
- net M2-: now also U5.7 (2A)
- net M2PWM: now also U5.1 (EN1,2)
- net SPK: now also J12.2 (Pin_2)
- net SRCLR: now also C8.1, D1.2 (A), R1.2
- net Vm: now also U4.8 (VCC2), U5.8 (VCC2)
- net at J14.1 (Pin_1): now also U4.6 (2Y)
- net at J16.2 (Pin_2): now also U5.3 (1Y)
- net at J14.2 (Pin_2): now also U4.3 (1Y)
- net at J16.1 (Pin_1): now also U5.6 (2Y)
- net at J15.1 (Pin_1): now also U4.14 (4Y)
- net at J15.2 (Pin_2): now also U4.11 (3Y)
- net Bump renamed Bump0
- net Bump0: no longer J8.2 (Pin_2)
- net MEnable renamed Bump1
- net Bump1: now also J8.2 (Pin_2)
- no-connect marks 8 -> 12
Other:
- moved on the sheet: U3

Commit message: did i finally figure out the motor drivers?
Parts:
- D1: footprint Diode_THT:D_DO-35_SOD27_P2.54mm_Vertical_AnodeUp -> Diode_THT:D_A-405_P7.62mm_Horizontal
- R2, R3, R4: footprint Resistors_THT:R_Axial_DIN0207_L6.3mm_D2.5mm_P7.62mm_Horizontal -> Resistor_THT:R_Axial_DIN0207_L6.3mm_D2.5mm_P7.62mm_Horizontal
Connections:
- net GND: no longer J10.2 (Pin_2), U4.12 (GND), U4.13 (GND), U4.4 (GND), U4.5 (GND), U5.12 (GND), U5.13 (GND), U5.4 (GND), U5.5 (GND)
- new net Gm: J10.2 (Pin_2), U4.12 (GND), U4.13 (GND), U4.4 (GND), U4.5 (GND), U5.12 (GND), U5.13 (GND), U5.4 (GND), U5.5 (GND)
Changed lines of the file:
@@
 F 0 "R3" V 6180 3450 50  0000 C CNN
 F 1 "R6" V 6100 3450 50  0000 C CNN
-F 2 "Resistors_THT:R_Axial_DIN0207_L6.3mm_D2.5mm_P7.62mm_Horizontal" V 6030 3450 50  0001 C CNN
+F 2 "Resistor_THT:R_Axial_DIN0207_L6.3mm_D2.5mm_P7.62mm_Horizontal" V 6030 3450 50  0001 C CNN
 F 3 "" H 6100 3450 50  0001 C CNN
 	1    6100 3450
@@
 F 0 "R2" V 5980 3450 50  0000 C CNN
 F 1 "R7" V 5900 3450 50  0000 C CNN
-F 2 "Resistors_THT:R_Axial_DIN0207_L6.3mm_D2.5mm_P7.62mm_Horizontal" V 5830 3450 50  0001 C CNN
+F 2 "Resistor_THT:R_Axial_DIN0207_L6.3mm_D2.5mm_P7.62mm_Horizontal" V 5830 3450 50  0001 C CNN
 F 3 "" H 5900 3450 50  0001 C CNN
 	1    5900 3450
@@
 F 0 "R4" V 6530 3850 50  0000 C CNN
 F 1 "R10" V 6450 3850 50  0000 C CNN
-F 2 "Resistors_THT:R_Axial_DIN0207_L6.3mm_D2.5mm_P7.62mm_Horizontal" V 6380 3850 50  0001 C CNN
+F 2 "Resistor_THT:R_Axial_DIN0207_L6.3mm_D2.5mm_P7.62mm_Horizontal" V 6380 3850 50  0001 C CNN
 F 3 "" H 6450 3850 50  0001 C CNN
 	1    6450 3850
@@
 	1500 5850 1800 5850
 Wire Wire Line
-	2200 6150 2450 6150
-Wire Wire Line
 	2850 6150 3200 6150
 Wire Wire Line
@@
 Wire Wire Line
 	3150 6850 3450 6850
-Wire Wire Line
-	3150 6950 3250 6950
 Text GLabel 3450 6850 2    50   Input ~ 0
 Vm
@@
 Text GLabel 3450 6950 2    50   Input ~ 0
 Gm
-Wire Wire Line
-	2450 6150 2450 7200
-Wire Wire Line
-	2450 7200 3250 7200
-Wire Wire Line
-	3250 7200 3250 6950
-Connection ~ 2450 6150
-Wire Wire Line
-	2450 6150 2850 6150
-Connection ~ 3250 6950
-Wire Wire Line
-	3250 6950 3450 6950
 $Comp
 L main_board-rescue:Conn_01x03_Male J3
@@
 F 0 "D1" V 4604 6705 50  0000 L CNN
 F 1 "D" V 4695 6705 50  0000 L CNN
-F 2 "Diode_THT:D_DO-35_SOD27_P2.54mm_Vertical_AnodeUp" H 4650 6625 50  0001 C CNN
+F 2 "Diode_THT:D_A-405_P7.62mm_Horizontal" H 4650 6625 50  0001 C CNN
 F 3 "~" H 4650 6625 50  0001 C CNN
 	1    4650 6625
@@
 Text GLabel 1200 5300 2    60   Input ~ 0
 9V
+Wire Wire Line
+	3150 6950 3450 6950
+Wire Wire Line
+	2200 6150 2850 6150
+$Comp
+L power:PWR_FLAG #FLG0102
+U 1 1 61D3D792
+P 3150 6950
+F 0 "#FLG0102" H 3150 7025 50  0001 C CNN
+F 1 "PWR_FLAG" H 3150 7123 50  0000 C CNN
+F 2 "" H 3150 6950 50  0001 C CNN
+F 3 "~" H 3150 6950 50  0001 C CNN
+	1    3150 6950
+	1    0    0    -1
+$EndComp
+Connection ~ 3150 6950
 $EndSCHEMATC
