File: tank/main_board/main_board.sch (KiCad schematic (older format))
At the start: 35 parts, among them J1 PowerOut, J10 PowerMotor, J11 SigOut, J12 Spk, J13 LEDs, J14 M0, J15 M1, J16 M2, J2 PowerIn, J3 Encoder0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

Commit message: fix serial register
Parts:
- U3: symbol custom:SN74HC595 -> main_board-rescue:SN74HC595-custom
Connections:
- net SER renamed SERIAL_DATA
- net SRCLK renamed SERIAL_CLOCK
- net SERIAL_CLOCK: no longer U3.12 (RCLK)
- net SRCLR: no longer names the net of C8.1, D1.2 (A), R1.2, U3.10 (SRCLR)
- net SRCLR: no longer U2.19 ((PCINT5/SCK)PB5)
- new net SERIAL_LATCH: U2.19 ((PCINT5/SCK)PB5)
Changed lines of the file:
@@
 	5250 6475 5200 6475
 Wire Wire Line
-	5200 6475 5200 6175
-Wire Wire Line
-	5100 6175 5200 6175
-Wire Wire Line
 	5250 6275 5125 6275
-Connection ~ 5200 6175
-Text GLabel 4400 6775 0    60   Input ~ 0
-SRCLR
 Text GLabel 5100 6175 0    60   Input ~ 0
-SRCLK
+SERIAL_CLOCK
 Text GLabel 5250 5975 0    60   Input ~ 0
-SER
+SERIAL_DATA
 Text GLabel 6650 5975 2    60   Input ~ 0
 M0+
@@
 Encoder0
 Text GLabel 5250 2400 2    60   Input ~ 0
-SER
+SERIAL_DATA
 Text GLabel 5250 2800 2    60   Input ~ 0
-SRCLK
+SERIAL_CLOCK
 Text GLabel 5250 2900 2    60   Input ~ 0
-SRCLR
+SERIAL_LATCH
 Text GLabel 5250 3250 2    60   Input ~ 0
 LED2
@@
 M2-
 $Comp
-L custom:SN74HC595 U3
+L main_board-rescue:SN74HC595-custom U3
 U 1 1 5A486ACA
 P 5950 6425
@@
 Wire Wire Line
 	6450 4000 6550 4000
-Wire Wire Line
-	5200 6175 5250 6175
 Wire Wire Line
 	6950 2900 6950 3200
@@
 $EndComp
 Connection ~ 3150 6950
+Wire Wire Line
+	5100 6175 5250 6175
+Text GLabel 5200 6450 0    50   Input ~ 0
+SERIAL_LATCH
 $EndSCHEMATC

Commit message: version 0.10 (i hate kicad library management with every fibre of my being)
Parts:
- C1, C3: footprint Capacitors_THT:CP_Radial_D4.0mm_P2.00mm -> Capacitor_THT:CP_Radial_D4.0mm_P2.00mm
- C4: footprint Capacitors_THT:C_Disc_D4.7mm_W2.5mm_P5.00mm -> Capacitor_THT:C_Disc_D4.7mm_W2.5mm_P5.00mm
- C5, C8: symbol Device:C_Small -> main_board-rescue:C_Small-Device
- D1: symbol Device:D -> main_board-rescue:D-Device
- J1, J10, J12, J2: footprint JST:JST_EH_B02B-EH-A_02x2.50mm_Straight -> Connector_JST:JST_EH_B2B-EH-A_1x02_P2.50mm_Vertical
- J11, J13: footprint JST:JST_EH_B04B-EH-A_04x2.50mm_Straight -> Connector_JST:JST_EH_B4B-EH-A_1x04_P2.50mm_Vertical
- J3, J4, J5, J6: footprint JST:JST_EH_B03B-EH-A_03x2.50mm_Straight -> Connector_JST:JST_EH_B3B-EH-A_1x03_P2.50mm_Vertical
- J9: footprint Pin_Headers:Pin_Header_Straight_1x06_Pitch2.54mm -> Connector_PinHeader_2.54mm:PinHeader_1x06_P2.54mm_Vertical
- R1: symbol Device:R -> main_board-rescue:R-Device
- U1: footprint Custom:L7805 -> Custom:L7805CV; symbol Regulator_Linear:L7805 -> main_board-rescue:L7805-Regulator_Linear
- U2: footprint Housings_DIP:DIP-28_W7.62mm_Socket -> Package_DIP:DIP-28_W7.62mm
- U3: footprint Housings_DIP:DIP-16_W7.62mm -> Package_DIP:DIP-16_W7.62mm
- U4, U5: symbol Driver_Motor:L293D -> main_board-rescue:L293D-Driver_Motor
- Y1: footprint Crystals:Crystal_HC49-U_Vertical -> Crystal:Crystal_HC49-U_Vertical
Connections:
- net SERIAL_LATCH: now also U3.12 (RCLK)
Other:
- moved on the sheet: C8, D1, R1
Changed lines of the file:
@@
 F 0 "U2" H 3500 4750 50  0000 L BNN
 F 1 "ATMEGA328P-PU" H 4650 2100 50  0000 L BNN
-F 2 "Housings_DIP:DIP-28_W7.62mm_Socket" H 4250 3500 50  0001 C CIN
+F 2 "Package_DIP:DIP-28_W7.62mm" H 4250 3500 50  0001 C CIN
 F 3 "" H 4250 3500 50  0001 C CNN
 	1    4250 3500
@@
 F 0 "C1" H 1525 5800 50  0000 L CNN
 F 1 "CP1" H 1525 5600 50  0000 L CNN
-F 2 "Capacitors_THT:CP_Radial_D4.0mm_P2.00mm" H 1538 5550 50  0001 C CNN
+F 2 "Capacitor_THT:CP_Radial_D4.0mm_P2.00mm" H 1538 5550 50  0001 C CNN
 F 3 "" H 1500 5700 50  0001 C CNN
 	1    1500 5700
@@
 F 0 "C3" H 2875 5800 50  0000 L CNN
 F 1 "CP3" H 2875 5600 50  0000 L CNN
-F 2 "Capacitors_THT:CP_Radial_D4.0mm_P2.00mm" H 2888 5550 50  0001 C CNN
+F 2 "Capacitor_THT:CP_Radial_D4.0mm_P2.00mm" H 2888 5550 50  0001 C CNN
 F 3 "" H 2850 5700 50  0001 C CNN
 	1    2850 5700
@@
 F 0 "Y1" H 6500 3200 50  0000 C CNN
 F 1 "Crystal" H 6500 2900 50  0000 C CNN
-F 2 "Crystals:Crystal_HC49-U_Vertical" H 6500 3050 50  0001 C CNN
+F 2 "Crystal:Crystal_HC49-U_Vertical" H 6500 3050 50  0001 C CNN
 F 3 "" H 6500 3050 50  0001 C CNN
 	1    6500 3050
@@
 F 0 "J11" H 3350 1250 50  0000 C CNN
 F 1 "SigOut" H 3350 750 50  0000 C CNN
-F 2 "JST:JST_EH_B04B-EH-A_04x2.50mm_Straight" H 3350 1050 50  0001 C CNN
+F 2 "Connector_JST:JST_EH_B4B-EH-A_1x04_P2.50mm_Vertical" H 3350 1050 50  0001 C CNN
 F 3 "" H 3350 1050 50  0001 C CNN
 	1    3350 1050
@@
 F 0 "C4" H 3260 4470 50  0000 L CNN
 F 1 "C4" H 3260 4320 50  0000 L CNN
-F 2 "Capacitors_THT:C_Disc_D4.7mm_W2.5mm_P5.00mm" H 3250 4400 50  0001 C CNN
+F 2 "Capacitor_THT:C_Disc_D4.7mm_W2.5mm_P5.00mm" H 3250 4400 50  0001 C CNN
 F 3 "" H 3250 4400 50  0001 C CNN
 	1    3250 4400
@@
 F 0 "J5" H 1850 2100 50  0000 C CNN
 F 1 "Encoder2" H 1850 1700 50  0000 C CNN
-F 2 "JST:JST_EH_B03B-EH-A_03x2.50mm_Straight" H 1850 1900 50  0001 C CNN
+F 2 "Connector_JST:JST_EH_B3B-EH-A_1x03_P2.50mm_Vertical" H 1850 1900 50  0001 C CNN
 F 3 "" H 1850 1900 50  0001 C CNN
 	1    1850 1900
@@
 F 0 "J6" H 1850 2450 50  0000 C CNN
 F 1 "Encoder3" H 1850 2050 50  0000 C CNN
-F 2 "JST:JST_EH_B03B-EH-A_03x2.50mm_Straight" H 1850 2250 50  0001 C CNN
+F 2 "Connector_JST:JST_EH_B3B-EH-A_1x03_P2.50mm_Vertical" H 1850 2250 50  0001 C CNN
 F 3 "" H 1850 2250 50  0001 C CNN
 	1    1850 2250
@@
 F 0 "J9" H 2200 4750 50  0000 C CNN
 F 1 "Programming Header" H 2200 4050 50  0000 C CNN
-F 2 "Pin_Headers:Pin_Header_Straight_1x06_Pitch2.54mm" H 2200 4450 50  0001 C CNN
+F 2 "Connector_PinHeader_2.54mm:PinHeader_1x06_P2.54mm_Vertical" H 2200 4450 50  0001 C CNN
 F 3 "" H 2200 4450 50  0001 C CNN
 	1    2200 4450
@@
 F 0 "J12" H 5300 850 50  0000 C CNN
 F 1 "Spk" H 5300 550 50  0000 C CNN
-F 2 "JST:JST_EH_B02B-EH-A_02x2.50mm_Straight" H 5300 750 50  0001 C CNN
+F 2 "Connector_JST:JST_EH_B2B-EH-A_1x02_P2.50mm_Vertical" H 5300 750 50  0001 C CNN
 F 3 "" H 5300 750 50  0001 C CNN
 	1    5300 750
@@
 F 0 "J1" H 700 4550 50  0000 C CNN
 F 1 "PowerOut" H 700 4250 50  0000 C CNN
-F 2 "JST:JST_EH_B02B-EH-A_02x2.50mm_Straight" H 700 4450 50  0001 C CNN
+F 2 "Connector_JST:JST_EH_B2B-EH-A_1x02_P2.50mm_Vertical" H 700 4450 50  0001 C CNN
 F 3 "" H 700 4450 50  0001 C CNN
 	1    700  4450
@@
 $EndComp
 $Comp
-L power:PWR_FLAG #FLG02
+L main_board-rescue:PWR_FLAG-power #FLG02
 U 1 1 59E6BC0C
 P 1350 5550
@@
 $EndComp
 $Comp
-L power:PWR_FLAG #FLG01
+L main_board-rescue:PWR_FLAG-power #FLG01
 U 1 1 59E6BD3A
 P 1200 5650
@@
 F 0 "J2" H 750 5650 50  0000 C CNN
 F 1 "PowerIn" H 750 5350 50  0000 C CNN
-F 2 "JST:JST_EH_B02B-EH-A_02x2.50mm_Straight" H 750 5550 50  0001 C CNN
+F 2 "Connector_JST:JST_EH_B2B-EH-A_1x02_P2.50mm_Vertical" H 750 5550 50  0001 C CNN
 F 3 "" H 750 5550 50  0001 C CNN
 	1    750  5550
@@
 IRRx
 $Comp
-L Regulator_Linear:L7805 U1
+L main_board-rescue:L7805-Regulator_Linear U1
 U 1 1 5A47F96E
 P 2200 5550
 F 0 "U1" H 2050 5675 50  0000 C CNN
 F 1 "L7805" H 2200 5675 50  0000 L CNN
-F 2 "Custom:L7805" H 2225 5400 50  0001 L CIN
+F 2 "Custom:L7805CV" H 2225 5400 50  0001 L CIN
 F 3 "" H 2200 5500 50  0001 C CNN
 	1    2200 5550
@@
 NoConn ~ 6650 6575
 NoConn ~ 6650 6675
-Text GLabel 5250 6575 0    60   Input ~ 0
-GND
-Wire Wire Line
-	5250 6475 5200 6475
-Wire Wire Line
-	5250 6275 5125 6275
-Text GLabel 5100 6175 0    60   Input ~ 0
+Text GLabel 5250 6175 0    60   Input ~ 0
 SERIAL_CLOCK
 Text GLabel 5250 5975 0    60   Input ~ 0
@@
 F 0 "U3" H 6100 7025 50  0000 C CNN
 F 1 "SN74HC595" H 5950 5825 50  0000 C CNN
-F 2 "Housings_DIP:DIP-16_W7.62mm" H 5950 6425 50  0001 C CNN
+F 2 "Package_DIP:DIP-16_W7.62mm" H 5950 6425 50  0001 C CNN
 F 3 "" H 5950 6425 50  0001 C CNN
 	1    5950 6425
 	1    0    0    -1
 $EndComp
-Text GLabel 4400 5800 0    60   Input ~ 0
-4.5V
-Text GLabel 4400 7050 0    60   Input ~ 0
+Text GLabel 4100 5800 0    60   Input ~ 0
+4.5V
+Text GLabel 4100 7050 0    60   Input ~ 0
 GND
 Wire Wire Line
@@
 F 0 "J10" H 2950 6950 50  0000 C CNN
 F 1 "PowerMotor" H 2950 6650 50  0000 C CNN
-F 2 "JST:JST_EH_B02B-EH-A_02x2.50mm_Straight" H 2950 6850 50  0001 C CNN
+F 2 "Connector_JST:JST_EH_B2B-EH-A_1x02_P2.50mm_Vertical" H 2950 6850 50  0001 C CNN
 F 3 "" H 2950 6850 50  0001 C CNN
 	1    2950 6850
@@
 F 0 "J3" H 1958 1381 50  0000 C CNN
 F 1 "Encoder0" H 1958 1290 50  0000 C CNN
-F 2 "JST:JST_EH_B03B-EH-A_03x2.50mm_Straight" H 1850 1100 50  0001 C CNN
+F 2 "Connector_JST:JST_EH_B3B-EH-A_1x03_P2.50mm_Vertical" H 1850 1100 50  0001 C CNN
 F 3 "" H 1850 1100 50  0001 C CNN
 	1    1850 1100
@@
 F 0 "J4" H 1958 1831 50  0000 C CNN
 F 1 "Encoder1" H 1958 1740 50  0000 C CNN
-F 2 "JST:JST_EH_B03B-EH-A_03x2.50mm_Straight" H 1850 1550 50  0001 C CNN
+F 2 "Connector_JST:JST_EH_B3B-EH-A_1x03_P2.50mm_Vertical" H 1850 1550 50  0001 C CNN
 F 3 "" H 1850 1550 50  0001 C CNN
 	1    1850 1550
@@
 F 0 "J13" H 5700 1900 50  0000 C CNN
 F 1 "LEDs" H 5700 1400 50  0000 C CNN
-F 2 "JST:JST_EH_B04B-EH-A_04x2.50mm_Straight" H 5700 1700 50  0001 C CNN
+F 2 "Connector_JST:JST_EH_B4B-EH-A_1x04_P2.50mm_Vertical" H 5700 1700 50  0001 C CNN
 F 3 "" H 5700 1700 50  0001 C CNN
 	1    5700 1700
@@
 	2650 5550 2850 5550
 $Comp
-L Device:C_Small C5
+L main_board-rescue:C_Small-Device C5
 U 1 1 61727AF7
 P 6550 4100
@@
 	6950 3200 6900 3200
 $Comp
-L Driver_Motor:L293D U4
+L main_board-rescue:L293D-Driver_Motor U4
 U 1 1 61A74B1D
 P 8950 1850
@@
 	9450 2050 9450 1950
 $Comp
-L Driver_Motor:L293D U5
+L main_board-rescue:L293D-Driver_Motor U5
 U 1 1 61B52F69
 P 9000 4400
@@
 M0PWM
 $Comp
-L Device:R R1
+L main_board-rescue:R-Device R1
 U 1 1 61C6B3C4
-P 4400 6625
-F 0 "R1" H 4470 6671 50  0000 L CNN
-F 1 "R" H 4470 6580 50  0000 L CNN
-F 2 "Resistor_THT:R_Axial_DIN0207_L6.3mm_D2.5mm_P7.62mm_Horizontal" V 4330 6625 50  0001 C CNN
-F 3 "~" H 4400 6625 50  0001 C CNN
-	1    4400 6625
+P 4100 6625
+F 0 "R1" H 4170 6671 50  0000 L CNN
+F 1 "R" H 4170 6580 50  0000 L CNN
+F 2 "Resistor_THT:R_Axial_DIN0207_L6.3mm_D2.5mm_P7.62mm_Horizontal" V 4030 6625 50  0001 C CNN
+F 3 "~" H 4100 6625 50  0001 C CNN
+	1    4100 6625
 	1    0    0    -1
 $EndComp
@@
 	5650 5875 5650 5800
 $Comp
-L Device:C_Small C8
+L main_board-rescue:C_Small-Device C8
 U 1 1 61C9FF1C
-P 4400 6875
-F 0 "C8" H 4492 6921 50  0000 L CNN
-F 1 "C_Small" H 4492 6830 50  0000 L CNN
-F 2 "Capacitor_THT:C_Disc_D4.7mm_W2.5mm_P5.00mm" H 4400 6875 50  0001 C CNN
-F 3 "~" H 4400 6875 50  0001 C CNN
-	1    4400 6875
-	1    0    0    -1
-$EndComp
-$Comp
-L Device:D D1
+P 4100 6875
+F 0 "C8" H 4192 6921 50  0000 L CNN
+F 1 "C_Small" H 4192 6830 50  0000 L CNN
+F 2 "Capacitor_THT:C_Disc_D4.7mm_W2.5mm_P5.00mm" H 4100 6875 50  0001 C CNN
+F 3 "~" H 4100 6875 50  0001 C CNN
+	1    4100 6875
+	1    0    0    -1
+$EndComp
+$Comp
+L main_board-rescue:D-Device D1
 U 1 1 61CA4DBE
-P 4650 6625
-F 0 "D1" V 4604 6705 50  0000 L CNN
-F 1 "D" V 4695 6705 50  0000 L CNN
-F 2 "Diode_THT:D_A-405_P7.62mm_Horizontal" H 4650 6625 50  0001 C CNN
-F 3 "~" H 4650 6625 50  0001 C CNN
-	1    4650 6625
+P 4350 6625
+F 0 "D1" V 4304 6705 50  0000 L CNN
+F 1 "D" V 4395 6705 50  0000 L CNN
+F 2 "Diode_THT:D_A-405_P7.62mm_Horizontal" H 4350 6625 50  0001 C CNN
+F 3 "~" H 4350 6625 50  0001 C CNN
+	1    4350 6625
 	0    1    1    0
 $EndComp
 Wire Wire Line
-	4400 6775 4650 6775
-Connection ~ 4400 6775
-Wire Wire Line
-	4650 6775 4950 6775
-Wire Wire Line
-	4950 6775 4950 6425
-Wire Wire Line
-	4950 6425 5125 6425
-Wire Wire Line
-	5125 6425 5125 6275
-Connection ~ 4650 6775
-Wire Wire Line
-	4400 6475 4400 5800
-Wire Wire Line
-	4400 5800 4650 5800
+	4100 6775 4350 6775
+Connection ~ 4100 6775
+Wire Wire Line
+	4100 6475 4100 5800
 Wire Wire Line
 	5650 6975 5650 7050
 Wire Wire Line
-	5650 7050 4400 7050
-Wire Wire Line
-	4400 6975 4400 7050
+	4100 6975 4100 7050
 NoConn ~ 6650 6875
-Wire Wire Line
-	4650 6475 4650 5800
-Connection ~ 4650 5800
-Wire Wire Line
-	4650 5800 5650 5800
 Text GLabel 8500 4200 0    60   Input ~ 0
 M2PWM
@@
 NoConn ~ 9200 4575
 $Comp
-L power:PWR_FLAG #FLG0101
+L main_board-rescue:PWR_FLAG-power #FLG0101
 U 1 1 61D3DF25
 P 3150 6850
@@
 	2200 6150 2850 6150
 $Comp
-L power:PWR_FLAG #FLG0102
+L main_board-rescue:PWR_FLAG-power #FLG0102
 U 1 1 61D3D792
 P 3150 6950
@@
 $EndComp
 Connection ~ 3150 6950
-Wire Wire Line
-	5100 6175 5250 6175
-Text GLabel 5200 6450 0    50   Input ~ 0
+Text GLabel 5250 6475 0    50   Input ~ 0
 SERIAL_LATCH
+Wire Wire Line
+	4350 6475 4350 5800
+Wire Wire Line
+	4100 5800 4350 5800
+Connection ~ 4350 5800
+Wire Wire Line
+	4350 5800 5650 5800
+Wire Wire Line
+	4575 6275 4575 6775
+Wire Wire Line
+	4575 6775 4350 6775
+Wire Wire Line
+	4575 6275 5250 6275
+Connection ~ 4350 6775
+Wire Wire Line
+	4100 7050 5250 7050
+Wire Wire Line
+	5250 6575 5250 7050
+Connection ~ 5250 7050
+Wire Wire Line
+	5250 7050 5650 7050
 $EndSCHEMATC

Commit message: I cannot believe that I screwed-up the Bump Sensor in such a dumb way and failed to run the design rule checker
Connections:
- net Bump1: now also J9.5 (Pin_5), U2.3 ((PCINT17/TXD)PD1); no longer U2.16 ((PCINT2/OC1B/~SS~)PB2)
- net Encoder3: now also U2.16 ((PCINT2/OC1B/~SS~)PB2); no longer J9.5 (Pin_5), U2.3 ((PCINT17/TXD)PD1)
Other:
- moved on the sheet: J3, J4, J5, J6
Changed lines of the file:
@@
 L main_board-rescue:Conn_01x03_Male J5
 U 1 1 59DDB019
-P 1850 1900
-F 0 "J5" H 1850 2100 50  0000 C CNN
-F 1 "Encoder2" H 1850 1700 50  0000 C CNN
-F 2 "Connector_JST:JST_EH_B3B-EH-A_1x03_P2.50mm_Vertical" H 1850 1900 50  0001 C CNN
-F 3 "" H 1850 1900 50  0001 C CNN
-	1    1850 1900
+P 1875 1850
+F 0 "J5" H 1875 2050 50  0000 C CNN
+F 1 "Encoder2" H 1875 1650 50  0000 C CNN
+F 2 "Connector_JST:JST_EH_B3B-EH-A_1x03_P2.50mm_Vertical" H 1875 1850 50  0001 C CNN
+F 3 "" H 1875 1850 50  0001 C CNN
+	1    1875 1850
 	1    0    0    -1
 $EndComp
@@
 L main_board-rescue:Conn_01x03_Male J6
 U 1 1 59DDB307
-P 1850 2250
-F 0 "J6" H 1850 2450 50  0000 C CNN
-F 1 "Encoder3" H 1850 2050 50  0000 C CNN
-F 2 "Connector_JST:JST_EH_B3B-EH-A_1x03_P2.50mm_Vertical" H 1850 2250 50  0001 C CNN
-F 3 "" H 1850 2250 50  0001 C CNN
-	1    1850 2250
+P 1875 2275
+F 0 "J6" H 1875 2475 50  0000 C CNN
+F 1 "Encoder3" H 1875 2075 50  0000 C CNN
+F 2 "Connector_JST:JST_EH_B3B-EH-A_1x03_P2.50mm_Vertical" H 1875 2275 50  0001 C CNN
+F 3 "" H 1875 2275 50  0001 C CNN
+	1    1875 2275
 	1    0    0    -1
 $EndComp
@@
 Wire Wire Line
 	3250 4500 3250 4600
-Wire Wire Line
-	2100 2000 2050 2000
 Wire Wire Line
 	6100 3600 6100 3650
@@
 L main_board-rescue:Conn_01x03_Male J3
 U 1 1 5E9F4FF5
-P 1850 1100
-F 0 "J3" H 1958 1381 50  0000 C CNN
-F 1 "Encoder0" H 1958 1290 50  0000 C CNN
-F 2 "Connector_JST:JST_EH_B3B-EH-A_1x03_P2.50mm_Vertical" H 1850 1100 50  0001 C CNN
-F 3 "" H 1850 1100 50  0001 C CNN
-	1    1850 1100
+P 1850 975
+F 0 "J3" H 1958 1256 50  0000 C CNN
+F 1 "Encoder0" H 1958 1165 50  0000 C CNN
+F 2 "Connector_JST:JST_EH_B3B-EH-A_1x03_P2.50mm_Vertical" H 1850 975 50  0001 C CNN
+F 3 "" H 1850 975 50  0001 C CNN
+	1    1850 975
 	1    0    0    -1
 $EndComp
@@
 L main_board-rescue:Conn_01x03_Male J4
 U 1 1 5EA0741C
-P 1850 1550
-F 0 "J4" H 1958 1831 50  0000 C CNN
-F 1 "Encoder1" H 1958 1740 50  0000 C CNN
-F 2 "Connector_JST:JST_EH_B3B-EH-A_1x03_P2.50mm_Vertical" H 1850 1550 50  0001 C CNN
-F 3 "" H 1850 1550 50  0001 C CNN
-	1    1850 1550
-	1    0    0    -1
-$EndComp
-Text GLabel 2050 1100 2    60   Input ~ 0
-4.5V
-Text GLabel 2050 1200 2    60   Input ~ 0
-GND
-Text GLabel 2050 1000 2    60   Input ~ 0
+P 1850 1475
+F 0 "J4" H 1958 1756 50  0000 C CNN
+F 1 "Encoder1" H 1958 1665 50  0000 C CNN
+F 2 "Connector_JST:JST_EH_B3B-EH-A_1x03_P2.50mm_Vertical" H 1850 1475 50  0001 C CNN
+F 3 "" H 1850 1475 50  0001 C CNN
+	1    1850 1475
+	1    0    0    -1
+$EndComp
+Text GLabel 2050 975  2    60   Input ~ 0
+4.5V
+Text GLabel 2050 1075 2    60   Input ~ 0
+GND
+Text GLabel 2050 875  2    60   Input ~ 0
 Encoder0
 $Comp
@@
 	1    0    0    -1
 $EndComp
-Text GLabel 5850 4400 2    50   Input ~ 0
-Encoder3
 Wire Wire Line
 	1700 4450 1700 5300
@@
 Wire Wire Line
 	6550 4200 6550 4950
-Text GLabel 2050 1550 2    60   Input ~ 0
-4.5V
-Text GLabel 2050 1650 2    60   Input ~ 0
-GND
-Text GLabel 2050 1450 2    60   Input ~ 0
+Text GLabel 2050 1475 2    60   Input ~ 0
+4.5V
+Text GLabel 2050 1575 2    60   Input ~ 0
+GND
+Text GLabel 2050 1375 2    60   Input ~ 0
 Encoder1
-Text GLabel 2050 1900 2    60   Input ~ 0
-4.5V
-Text GLabel 2050 2000 2    60   Input ~ 0
-GND
-Text GLabel 2050 1800 2    60   Input ~ 0
+Text GLabel 2075 1850 2    60   Input ~ 0
+4.5V
+Text GLabel 2075 1950 2    60   Input ~ 0
+GND
+Text GLabel 2075 1750 2    60   Input ~ 0
 Encoder2
-Text GLabel 2050 2250 2    60   Input ~ 0
-4.5V
-Text GLabel 2050 2350 2    60   Input ~ 0
-GND
-Text GLabel 2050 2150 2    60   Input ~ 0
+Text GLabel 2075 2275 2    60   Input ~ 0
+4.5V
+Text GLabel 2075 2375 2    60   Input ~ 0
+GND
+Text GLabel 2075 2175 2    60   Input ~ 0
 Encoder3
 $Comp
@@
 M2PWM
 Text GLabel 5250 2600 2    50   Input ~ 0
-Bump1
+Encoder3
 NoConn ~ 8500 4800
 NoConn ~ 10075 -325
@@
 Wire Wire Line
 	5250 7050 5650 7050
+Text GLabel 5850 4400 2    50   Input ~ 0
+Bump1
 $EndSCHEMATC

Commit message: Major cleanup. I localized all the footprint and symbol libraries.
I deleted most of the rescue stuff.

I still need to finish-up changes to the turret board.

Now this checkout should work "out of the box".
Parts:
- C1, C3: footprint Capacitor_THT:CP_Radial_D4.0mm_P2.00mm -> custom:CP_Radial_D4.0mm_P2.00mm; symbol main_board-rescue:CP -> custom:CP
- C2: footprint Capacitor_THT:C_Disc_D4.7mm_W2.5mm_P5.00mm -> custom:C_Disc_D4.7mm_W2.5mm_P5.00mm; symbol main_board-rescue:C -> custom:C
- C4, C6, C7: footprint Capacitor_THT:C_Disc_D4.7mm_W2.5mm_P5.00mm -> custom:C_Disc_D4.7mm_W2.5mm_P5.00mm; symbol main_board-rescue:C_Small -> custom:C_Small
- C5, C8: footprint Capacitor_THT:C_Disc_D4.7mm_W2.5mm_P5.00mm -> custom:C_Disc_D4.7mm_W2.5mm_P5.00mm; symbol main_board-rescue:C_Small-Device -> custom:C_Small-Device
- D1: footprint Diode_THT:D_A-405_P7.62mm_Horizontal -> custom:D_A-405_P7.62mm_Horizontal; symbol main_board-rescue:D-Device -> custom:D-Device
- J1, J10, J12, J14, J15, J16, J2, J7, J8: footprint Connector_JST:JST_EH_B2B-EH-A_1x02_P2.50mm_Vertical -> custom:JST_EH_B2B-EH-A_1x02_P2.50mm_Vertical; symbol main_board-rescue:Conn_01x02_Male -> custom:Conn_01x02_Male
- J11, J13: footprint Connector_JST:JST_EH_B4B-EH-A_1x04_P2.50mm_Vertical -> custom:JST_EH_B4B-EH-A_1x04_P2.50mm_Vertical; symbol main_board-rescue:Conn_01x04_Male -> custom:Conn_01x04_Male
- J3, J4, J5, J6: footprint Connector_JST:JST_EH_B3B-EH-A_1x03_P2.50mm_Vertical -> custom:JST_EH_B3B-EH-A_1x03_P2.50mm_Vertical; symbol main_board-rescue:Conn_01x03_Male -> custom:Conn_01x03_Male
- J9: footprint Connector_PinHeader_2.54mm:PinHeader_1x06_P2.54mm_Vertical -> custom:PinHeader_1x06_P2.54mm_Vertical; symbol main_board-rescue:Conn_01x06_Male -> custom:Conn_01x06_Male
- R1: footprint Resistor_THT:R_Axial_DIN0207_L6.3mm_D2.5mm_P7.62mm_Horizontal -> custom:R_Axial_DIN0207_L6.3mm_D2.5mm_P7.62mm_Horizontal; symbol main_board-rescue:R-Device -> custom:R-Device
- R2, R3, R4: footprint Resistor_THT:R_Axial_DIN0207_L6.3mm_D2.5mm_P7.62mm_Horizontal -> custom:R_Axial_DIN0207_L6.3mm_D2.5mm_P7.62mm_Horizontal; symbol main_board-rescue:R -> custom:R
- U1: symbol main_board-rescue:L7805-Regulator_Linear -> custom:L7805-Regulator_Linear
- U2: footprint Package_DIP:DIP-28_W7.62mm -> custom:DIP-28_W7.62mm; symbol main_board-rescue:ATMEGA328P-PU -> custom:ATMEGA328P-PU
- U3: footprint Package_DIP:DIP-16_W7.62mm -> custom:DIP-16_W7.62mm; symbol main_board-rescue:SN74HC595-custom -> custom:SN74HC595-custom
- U4, U5: footprint Package_DIP:DIP-16_W7.62mm -> custom:DIP-16_W7.62mm; symbol main_board-rescue:L293D-Driver_Motor -> custom:L293D-Driver_Motor
- Y1: symbol main_board-rescue:Crystal -> custom:Crystal
