File: tank/bump_sensor/bump_sensor.sch (KiCad schematic (older format))
At the start: 3 parts, among them J1 Conn_01x02_Male, SW1 SW_SPDT, SW2 SW_SPDT

Commit message: Major cleanup. I localized all the footprint and symbol libraries.
I deleted most of the rescue stuff.

I still need to finish-up changes to the turret board.

Now this checkout should work "out of the box".
Parts:
- J1: footprint (none) -> custom:JST_EH_B2B-EH-A_1x02_P2.50mm_Vertical; symbol Connector:Conn_01x02_Male -> custom:Conn_01x02_Male
- SW1, SW2: footprint (none) -> custom:micro_switch; symbol Switch:SW_SPDT -> custom:SW_SPDT
Changed lines of the file:
@@
 $EndDescr
 $Comp
-L Switch:SW_SPDT SW1
+L custom:SW_SPDT SW1
 U 1 1 615E113B
 P 4000 3400
 F 0 "SW1" H 4000 3685 50  0000 C CNN
 F 1 "SW_SPDT" H 4000 3594 50  0000 C CNN
-F 2 "" H 4000 3400 50  0001 C CNN
+F 2 "custom:micro_switch" H 4000 3400 50  0001 C CNN
 F 3 "~" H 4000 3400 50  0001 C CNN
 	1    4000 3400
@@
 $EndComp
 $Comp
-L Connector:Conn_01x02_Male J1
+L custom:Conn_01x02_Male J1
 U 1 1 615E2518
 P 2800 3600
 F 0 "J1" H 2908 3781 50  0000 C CNN
 F 1 "Conn_01x02_Male" H 2908 3690 50  0000 C CNN
-F 2 "" H 2800 3600 50  0001 C CNN
+F 2 "custom:JST_EH_B2B-EH-A_1x02_P2.50mm_Vertical" H 2800 3600 50  0001 C CNN
 F 3 "~" H 2800 3600 50  0001 C CNN
 	1    2800 3600
@@
 $EndComp
 $Comp
-L Switch:SW_SPDT SW2
+L custom:SW_SPDT SW2
 U 1 1 615E31A3
 P 4000 3950
 F 0 "SW2" H 4000 4235 50  0000 C CNN
 F 1 "SW_SPDT" H 4000 4144 50  0000 C CNN
-F 2 "" H 4000 3950 50  0001 C CNN
+F 2 "custom:micro_switch" H 4000 3950 50  0001 C CNN
 F 3 "~" H 4000 3950 50  0001 C CNN
 	1    4000 3950
