File: tank_trainer/tank_trainer.kicad_pcb (KiCad board)
At the start: 2 copper layers, 33 x 52 mm, 20 parts, among them U1 L7805, U2 ATMEGA328P-PU, Y1 Crystal

Commit message: update tank trainer to add programming header
Parts:
- removed PowerIn: PowerIn, Connector_JST:JST_EH_B2B-EH-A_1x02_P2.50mm_Vertical
- added C5: 100nF, Capacitor_THT:C_Disc_D5.0mm_W2.5mm_P2.50mm, F.Cu at (54.1, 89.2)
- added PowerIn1: PowerIn, Connector_JST:JST_EH_B2B-EH-A_1x02_P2.50mm_Vertical, F.Cu at (67.6, 74.4)
- added ProgrammingHeader1: Programming Header, Connector_PinHeader_2.54mm:PinHeader_1x06_P2.54mm_Horizontal, F.Cu at (49.5, 99.6)
- added R4: R, Resistor_THT:R_Axial_DIN0207_L6.3mm_D2.5mm_P7.62mm_Horizontal, F.Cu at (54.1, 100.1)
- moved Beacon1 24.5 mm to (41.9, 106.4), turned to -90 degrees
- moved U1 21.1 mm to (48.7, 73.9), turned to 0 degrees
- moved C3 14.0 mm to (53.8, 80.0)
- moved C1 9.03 mm to (48.8, 80.0)
- moved C2 8.72 mm to (60.0, 79.5)
- moved H4 7.40 mm to (42.4, 118.6)
- moved H1 6.63 mm to (42.4, 77.2)
- moved H5 3.51 mm to (74.9, 118.6)
- moved C7 3.50 mm to (50.6, 119.1)
- moved Y1 3.47 mm to (51.8, 114.0)
- moved C6 2.86 mm to (50.6, 103.4)
- moved H3 0.89 mm to (74.4, 77.2)
Connections:
- net 9V renamed Net-(PowerIn1-Pin_1)
- net Net-(LED0-Pin_2) renamed Rx
- U2 pad 1: 4.5V -> Net-(U2-(PCINT14/~{RESET})PC6)
- U2 pad 20: 4.5V -> unconnected-(U2-AVCC-Pad20)
- U2 pad 3: unconnected-(U2-(PCINT17/TXD)PD1-Pad3) -> Tx
Routing:
- net Rx: track 5.26 -> 29.2 mm
- net Net-(Beacon1-Pin_2): track 11.7 -> 32.6 mm
- net Net-(U2-(PCINT14/~{RESET})PC6): track 0.00 -> 11.4 mm
- net GND: track 110.1 -> 120.8 mm
- net Tx: track 0.00 -> 9.04 mm
- net 4.5V: track 53.9 -> 60.6 mm
- net Net-(ProgrammingHeader1-Pin_6): track 0.00 -> 5.52 mm
- net Net-(PowerIn1-Pin_1): track 23.0 -> 26.6 mm
- net Net-(IRRx1-Pin_1): track 26.4 -> 29.0 mm
- net Net-(U2-(PCINT7/XTAL2/TOSC2)PB7): track 14.9 -> 15.4 mm
- net Net-(U2-(PCINT6/XTAL1/TOSC1)PB6): track 14.0 -> 14.5 mm
Other:
- board size 33 x 52 mm -> 39.3 x 50.7 mm

Commit message: tank trainer v0.2 (whoops ... forgot the button)
Parts:
- added Button1: Conn_01x02_Pin, Connector_JST:JST_EH_B2B-EH-A_1x02_P2.50mm_Vertical, F.Cu at (64.0, 122.2)
- moved H5 3.66 mm to (73.4, 121.9)
- moved H4 3.30 mm to (42.4, 121.9)
- moved H3 2.06 mm to (73.3, 75.5)
- moved PowerIn1 1.71 mm to (66.0, 75.1)
- moved H1 1.68 mm to (42.4, 75.5)
- moved Beacon1 0.59 mm to (41.6, 105.9)
Connections:
- U2 pad 4: unconnected-(U2-(PCINT18/INT0)PD2-Pad4) -> Net-(Button1-Pin_2)
Other:
- board size 39.3 x 50.7 mm -> 37.7 x 52.9 mm
- board text added: "Laser Tag Robot Tank Tank Trainer v0.2"
- board text removed: "Laser Tag Robot Tank Tank Trainer v0.1"

Commit message: minor changes for turret board v0.11
Connections:
- Button1 pad 1: (no net) -> GND
- Button1 pad 2: (no net) -> Net-(Button1-Pin_2)
Routing:
- net Net-(Button1-Pin_2): track 0.00 -> 34.4 mm
- net GND: track 120.8 -> 152.8 mm
- net Net-(PowerIn1-Pin_1): track 26.6 -> 23.0 mm
- net 4.5V: track 60.6 -> 62.3 mm
Other:
- board text added: "Laser Tag Robot Tank Tank Trainer v0.3"
- board text removed: "Laser Tag Robot Tank Tank Trainer v0.2"
Changed lines of the file:
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@@
 			)
 		)
+		(property ki_fp_filters "Connector*:*_1x??_*")
+		(sheetname "/")
+		(sheetfile "tank_trainer.kicad_sch")
 		(attr through_hole)
 		(fp_line
@@
 			(remove_unused_layers no)
 			(roundrect_rratio 0.147059)
+			(net 1 "GND")
 			(pinfunction "Pin_1")
 			(pintype "passive")
@@
 			(layers "*.Cu" "*.Mask")
 			(remove_unused_layers no)
+			(net 23 "Net-(Button1-Pin_2)")
 			(pinfunction "Pin_2")
 			(pintype "passive")
@@
 			)
 		)
+		(property ki_fp_filters "MountingHole*")
+		(sheetname "/")
+		(sheetfile "tank_trainer.kicad_sch")
 		(attr exclude_from_pos_files exclude_from_bom)
 		(fp_circle
@@
 		(layer "Edge.Cuts")
 	)
-	(gr_text "Laser Tag Robot Tank\nTank Trainer v0.2"
+	(gr_text "Laser Tag Robot Tank\nTank Trainer v0.3"
 		(at 63 85 90)
 		(layer "B.SilkS")
@@
 	)
 	(segment
-		(start 62.74 101.61)
-		(end 65.28 99.07)
+		(start 65.6488 123.9012)
+		(end 63.9772 122.2296)
+		(width 0.2)
+		(layer "F.Cu")
+		(net 1)
+	)
+	(segment
+		(start 67.6282 123.2782)
+		(end 67.0052 123.9012)
 		(width 0.2)
 		(layer "F.Cu")
@@
 	)
 	(segment
-		(start 74 98.5)
-		(end 75.276 99.776)
+		(start 63.4892 78.4968)
+		(end 62.484 79.502)
 		(width 0.2)
 		(layer "F.Cu")
@@
 	)
 	(segment
-		(start 65.064 74.422)
-		(end 65.064 76.922)
+		(start 74 98.5)
+		(end 75.276 99.776)
 		(width 0.2)
 		(layer "F.Cu")
@@
 	)
 	(segment
+		(start 67.6282 101.4182)
+		(end 67.6282 123.2782)
+		(width 0.2)
+		(layer "F.Cu")
+		(net 1)
+	)
+	(segment
 		(start 62.484 79.502)
 		(end 66.002 79.502)
@@
 	)
 	(segment
-		(start 57.66 101.61)
-		(end 62.74 101.61)
+		(start 67.0052 123.9012)
+		(end 65.6488 123.9012)
 		(width 0.2)
 		(layer "F.Cu")
@@
 	)
 	(segment
-		(start 65.064 76.922)
-		(end 62.484 79.502)
+		(start 65.28 99.07)
+		(end 67.6282 101.4182)
+		(width 0.2)
+		(layer "F.Cu")
+		(net 1)
+	)
+	(segment
+		(start 63.4892 75.0824)
+		(end 63.4892 78.4968)
 		(width 0.2)
 		(layer "F.Cu")
@@
 	)
 	(segment
+		(start 60.8736 119.126)
+		(end 63.9772 122.2296)
+		(width 0.2)
+		(layer "B.Cu")
+		(net 1)
+	)
+	(segment
 		(start 49.53 99.822)
 		(end 53.086 103.378)
@@
 	)
 	(segment
+		(start 53.066 119.126)
+		(end 60.8736 119.126)
+		(width 0.2)
+		(layer "B.Cu")
+		(net 1)
+	)
+	(segment
 		(start 55.848 80.01)
 		(end 56.448 80.61)
@@
 	)
 	(segment
-		(start 54.899 74.842)
-		(end 53.848 75.893)
-		(width 0.2)
-		(layer "F.Cu")
-		(net 3)
-	)
-	(segment
-		(start 53.848 75.893)
-		(end 53.848 80.01)
+		(start 59.184001 78.702001)
+		(end 59.984 79.502)
 		(width 0.2)
-		(layer "F.Cu")
+		(layer "B.Cu")
 		(net 3)
 	)
@@
 	)
 	(segment
+		(start 55.155999 78.702001)
+		(end 59.184001 78.702001)
+		(width 0.2)
+		(layer "B.Cu")
+		(net 3)
+	)
+	(segment
 		(start 74 107)
 		(end 69.62 107)
@@
 	)
 	(segment
-		(start 59.591 79.109)
-		(end 59.984 79.502)
+		(start 59.984 79.502)
+		(end 55.324 74.842)
 		(width 0.2)
 		(layer "B.Cu")
@@
 	)
 	(segment
-		(start 54.749 79.109)
-		(end 59.591 79.109)
-		(width 0.2)
-		(layer "B.Cu")
-		(net 3)
-	)
-	(segment
 		(start 56.654 100.076)
 		(end 57.66 99.07)
@@
 	(segment
 		(start 53.848 80.01)
-		(end 54.749 79.109)
+		(end 55.155999 78.702001)
+		(width 0.2)
+		(layer "B.Cu")
+		(net 3)
+	)
+	(segment
+		(start 55.324 74.842)
+		(end 54.899 74.842)
 		(width 0.2)
 		(layer "B.Cu")
@@
 	)
 	(segment
+		(start 58.761 92.551)
+		(end 58.761 114.5134)
+		(width 0.2)
+		(layer "F.Cu")
+		(net 23)
+	)
+	(segment
+		(start 57.66 91.45)
+		(end 58.761 92.551)
+		(width 0.2)
+		(layer "F.Cu")
+		(net 23)
+	)
+	(segment
+		(start 58.761 114.5134)
+		(end 66.4772 122.2296)
+		(width 0.2)
+		(layer "F.Cu")
+		(net 23)
+	)
+	(segment
 		(start 55.203 91.355)
 		(end 54.102 92.456)
@@
 	)
 	(segment
-		(start 50.292 78.518)
-		(end 48.8 80.01)
-		(width 0.2)
-		(layer "B.Cu")
-		(net 31)
-	)
-	(segment
-		(start 59.41095 78.518)
-		(end 50.292 78.518)
+		(start 48.8 75.721)
+		(end 49.679 74.842)
 		(width 0.2)
-		(layer "B.Cu")
-		(net 31)
-	)
-	(segment
-		(start 49.679 74.842)
-		(end 49.679 79.131)
-		(width 0.2)
-		(layer "B.Cu")
+		(layer "F.Cu")
 		(net 31)
 	)
 	(segment
-		(start 67.564 74.422)
-		(end 66.00695 75.97905)
+		(start 48.8 80.01)
+		(end 48.8 75.721)
 		(width 0.2)
-		(layer "B.Cu")
+		(layer "F.Cu")
 		(net 31)
 	)
 	(segment
-		(start 66.00695 75.97905)
-		(end 61.9499 75.97905)
+		(start 51.01 73.511)
+		(end 49.679 74.842)
 		(width 0.2)
 		(layer "B.Cu")
@@
 	)
 	(segment
-		(start 61.9499 75.97905)
-		(end 59.41095 78.518)
+		(start 65.9892 75.0824)
+		(end 64.4178 73.511)
 		(width 0.2)
 		(layer "B.Cu")
@@
 	)
 	(segment
-		(start 49.679 79.131)
-		(end 48.8 80.01)
+		(start 64.4178 73.511)
+		(end 51.01 73.511)
 		(width 0.2)
 		(layer "B.Cu")

Commit message: Main Board v0.17 Tank Trainer v0.3
Parts:
- removed C7: 22pF, Capacitor_THT:C_Disc_D5.0mm_W2.5mm_P2.50mm
- removed H5: MountingHole, MountingHole:MountingHole_3mm
- removed LED0: Conn_01x02_Pin, Connector_JST:JST_EH_B2B-EH-A_1x02_P2.50mm_Vertical
- added C4: 22pF, Capacitor_THT:C_Disc_D5.0mm_W2.5mm_P2.50mm, F.Cu at (50.6, 118.0)
- added G***: LOGO, custom:Tank, B.Cu at (46.9, 102.7)
- added H2: MountingHole, MountingHole:MountingHole_3mm, F.Cu at (73.4, 121.8)
- added LED1: Conn_01x02_Pin, Connector_JST:JST_EH_B2B-EH-A_1x02_P2.50mm_Vertical, F.Cu at (74.0, 88.2)
- added LED2: Conn_01x02_Pin, Connector_JST:JST_EH_B2B-EH-A_1x02_P2.50mm_Vertical, F.Cu at (63.6, 123.0)
- added R5: R, Resistor_THT:R_Axial_DIN0207_L6.3mm_D2.5mm_P7.62mm_Horizontal, F.Cu at (68.5, 90.9)
- C5: value 100nF -> 22pF
- C6: value 22pF -> 100nF
- moved R1 33.7 mm to (46.5, 117.1)
- moved R4 26.5 mm to (68.5, 122.3)
- moved Button1 12.2 mm to (51.8, 122.5)
- moved R2 2.10 mm to (68.5, 104.3)
- moved R3 1.33 mm to (68.5, 101.4)
- moved Y1 1.03 mm to (51.8, 112.9)
- moved C6 0.41 mm to (50.6, 103.0)
- moved H4 0.16 mm to (42.4, 121.8)
Connections:
- C5 pad 1: Net-(ProgrammingHeader1-Pin_6) -> Net-(U2-(PCINT7/XTAL2/TOSC2)PB7)
- C5 pad 2: Net-(U2-(PCINT14/~{RESET})PC6) -> GND
- C6 pad 1: Net-(U2-(PCINT6/XTAL1/TOSC1)PB6) -> Net-(ProgrammingHeader1-Pin_6)
- C6 pad 2: GND -> Net-(U2-(PCINT14/~{RESET})PC6)
- R1 pad 1: Net-(U2-(PCINT16/RXD)PD0) -> 4.5V
- R1 pad 2: Rx -> Net-(Beacon1-Pin_2)
- R2 pad 1: 4.5V -> Net-(U2-(PCINT9/ADC1)PC1)
- R2 pad 2: Net-(Beacon1-Pin_2) -> Net-(IRTx1-Pin_2)
- R3 pad 1: Net-(U2-(PCINT9/ADC1)PC1) -> Net-(U2-(PCINT1/OC1A)PB1)
- R3 pad 2: Net-(IRTx1-Pin_2) -> Net-(LED1-Pin_2)
- R4 pad 1: 4.5V -> Net-(U2-(PCINT22/OC0A/AIN0)PD6)
- R4 pad 2: Net-(U2-(PCINT14/~{RESET})PC6) -> Net-(LED2-Pin_2)
- U2 pad 12: unconnected-(U2-(PCINT22/OC0A/AIN0)PD6-Pad12) -> Net-(U2-(PCINT22/OC0A/AIN0)PD6)
- U2 pad 15: unconnected-(U2-(PCINT1/OC1A)PB1-Pad15) -> Net-(U2-(PCINT1/OC1A)PB1)
- U2 pad 2: Net-(U2-(PCINT16/RXD)PD0) -> Rx
Routing:
- net 4.5V: track 62.3 -> 134.7 mm
- net Net-(Beacon1-Pin_2): track 32.6 -> 5.31 mm
- net Net-(U2-(PCINT22/OC0A/AIN0)PD6): track 0.00 -> 25.6 mm
- net Net-(U2-(PCINT14/~{RESET})PC6): track 11.4 -> 34.6 mm
- net GND: track 152.8 -> 132.9 mm
- net Net-(U2-(PCINT1/OC1A)PB1): track 0.00 -> 16.8 mm
- net Rx: track 29.2 -> 13.8 mm
- net Net-(U2-(PCINT16/RXD)PD0): track 13.7 -> 0.00 mm
- net Net-(IRTx1-Pin_2): track 5.41 -> 18.3 mm
- net Net-(U2-(PCINT7/XTAL2/TOSC2)PB7): track 15.4 -> 28.2 mm
- net Net-(LED2-Pin_2): track 0.00 -> 11.4 mm
- net Net-(ProgrammingHeader1-Pin_6): track 5.52 -> 16.6 mm
- net Net-(LED1-Pin_2): track 0.00 -> 10.3 mm
- net Net-(IRRx1-Pin_1): track 29.0 -> 37.5 mm
- net Net-(U2-(PCINT6/XTAL1/TOSC1)PB6): track 14.5 -> 17.8 mm
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