File: tank_trainer/tank_trainer.kicad_sch (KiCad schematic)
At the start: 20 parts, among them J9 PowerIn, U1 L7805, U2 ATMEGA328P-PU, Y1 Crystal

Commit message: update tank trainer to add programming header
Parts:
- added C5: 100nF, Capacitor_THT:C_Disc_D5.0mm_W2.5mm_P2.50mm, symbol Device:C_Small
- added ProgrammingHeader1: Programming Header, Connector_PinHeader_2.54mm:PinHeader_1x06_P2.54mm_Horizontal, symbol Connector:Conn_01x06_Pin
- added R4: R, Resistor_THT:R_Axial_DIN0207_L6.3mm_D2.5mm_P7.62mm_Horizontal, symbol Device:R
- renumbered J9 to PowerIn1
Connections:
- net 4.5V: now also ProgrammingHeader1.3 (Pin_3), R4.1; no longer U2.1 ((PCINT14/~{RESET})PC6), U2.20 (AVCC)
- net GND: now also ProgrammingHeader1.1 (Pin_1)
- net Rx: now reaches LED0.2 (Pin_2), R1.2
- net Rx: now also ProgrammingHeader1.4 (Pin_4)
- net Tx: now reaches U2.3 ((PCINT17/TXD)PD1)
- net Tx: now also ProgrammingHeader1.5 (Pin_5)
- net 9V: no longer names the net of C1.1, PowerIn1.1 (Pin_1), U1.1 (IN)
- new net: C5.2, R4.2, U2.1 ((PCINT14/~{RESET})PC6)
- new net: C5.1, ProgrammingHeader1.6 (Pin_6)
- no-connect marks 18 -> 19
Other:
- moved on the sheet: Beacon1, C1, C2, H3, IRTx1, PowerIn1, R2, R3

Commit message: tank trainer v0.2 (whoops ... forgot the button)
Parts:
- added Button: Conn_01x02_Pin, Connector_JST:JST_EH_B2B-EH-A_1x02_P2.50mm_Vertical, symbol Connector:Conn_01x02_Pin
Connections:
- net GND: now also Button.1 (Pin_1)
- net at U2.4 ((PCINT18/INT0)PD2): now also Button.2 (Pin_2)
- no-connect marks 19 -> 18
Other:
- moved on the sheet: C5, IRTx1, R4

Commit message: minor changes for turret board v0.11
Parts:
- renumbered Button to Button1
Changed lines of the file:
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@@
 		(dnp no)
 		(fields_autoplaced yes)
-		(property "Reference" "Button"
+		(property "Reference" "Button1"
 			(at 186.69 82.5499 0)
 			(effects
@@
 			(project "tank_trainer"
 				(path "/bbdf6b73-423d-4868-8bf7-eea4b49abb4e"
-					(reference "Button")
+					(reference "Button1")
 					(unit 1)
 				)

Commit message: Main Board v0.17 Tank Trainer v0.3
Parts:
- added LED2: Conn_01x02_Pin, Connector_JST:JST_EH_B2B-EH-A_1x02_P2.50mm_Vertical, symbol Connector:Conn_01x02_Pin
- added R4: R, Resistor_THT:R_Axial_DIN0207_L6.3mm_D2.5mm_P7.62mm_Horizontal, symbol Device:R
- renumbered C6 to C4, C7 to C5, C5 to C6, H4 to H1, H1 to H2, H5 to H3, H3 to H4, LED0 to LED1, R2 to R1, R3 to R2, R1 to R3, R4 to R5
Connections:
- net 4.5V: now also LED1.1 (Pin_1), LED2.1 (Pin_1)
- net GND: no longer LED1.1 (Pin_1)
- net Rx: now also U2.2 ((PCINT16/RXD)PD0); no longer LED1.2 (Pin_2), R3.2
- net at R3.1: now also U2.15 ((PCINT1/OC1A)PB1); no longer U2.2 ((PCINT16/RXD)PD0)
- net at U2.12 ((PCINT22/OC0A/AIN0)PD6): now also R4.1
- new net: LED2.2 (Pin_2), R4.2
- new net: LED1.2 (Pin_2), R3.2
- no-connect marks 18 -> 16
Other:
- moved on the sheet: Beacon1, LED1, R1, R3
